File: bipolar_input_opamp_style_power_amp_100W/bipolar_input_opamp_style_power_amp.kicad_pcb (KiCad board)
At the start: 2 copper layers, 34.3 x 31 mm, 33 parts, among them J1 IN+, J2 IN-, J3 VCC, J4 VEE, J5 OUT, J6 GND, Q1 MMDT5401, Q11 PZTA42-QX, Q12 PZTA92-QX, Q13 MJD31CG, Q14 MJD32CG, Q2 MMDT5551, Q3 MMDT5551, Q4 MMDT5401, Q5 MMDT5401, Q6 MMDT5551, Q7 PZTA92-QX, Q8 PZTA42-QX

Commit message: Add files via upload
Parts:
- removed REF** (x4): MountingHole_2.2mm_M2_ISO7380_Pad, MountingHole:MountingHole_2.2mm_M2_ISO7380_Pad
- removed RN1, RN2: 4x560R, Resistor_SMD:R_Array_Convex_4x1206
- added J7: GNDOUT, misc:726386-2, F.Cu at (186.4, 104.1)
- added J8: +IN, misc:SMA6251A13GT50G50, F.Cu at (90.8, 97.6)
- added Q10: PZTA92-QX, Package_TO_SOT_SMD:SOT-223, B.Cu at (132.1, 127.5)
- added Q15: MJD32C, PCM_Package_TO_SOT_SMD_AKL:TO-252-2, B.Cu at (172.3, 124.8)
- added Q16: MJD32C, PCM_Package_TO_SOT_SMD_AKL:TO-252-2, B.Cu at (162.2, 124.8)
- added Q17: MJD32C, PCM_Package_TO_SOT_SMD_AKL:TO-252-2, B.Cu at (152.0, 124.8)
- added Q18: MJD32C, PCM_Package_TO_SOT_SMD_AKL:TO-252-2, B.Cu at (141.9, 124.8)
- added Q19: PZTA92-QX, Package_TO_SOT_SMD:SOT-223, B.Cu at (132.1, 119.9)
- added Q20: PZTA42-QX, Package_TO_SOT_SMD:SOT-223, B.Cu at (132.1, 108.7)
- added Q9: PZTA42-QX, Package_TO_SOT_SMD:SOT-223, B.Cu at (132.1, 101.1)
- added R10: 47R, Resistor_SMD:R_0805_2012Metric_Pad1.20x1.40mm_HandSolder, F.Cu at (96.8, 131.8)
- added R11: 47R, Resistor_SMD:R_0805_2012Metric_Pad1.20x1.40mm_HandSolder, F.Cu at (101.5, 120.0)
- added R12: 100R, Resistor_SMD:R_0805_2012Metric_Pad1.20x1.40mm_HandSolder, F.Cu at (101.5, 122.9)
- added R13: GAIN, Resistor_SMD:R_0805_2012Metric_Pad1.20x1.40mm_HandSolder, F.Cu at (101.5, 125.9)
- added R14: 1k, Resistor_SMD:R_0805_2012Metric_Pad1.20x1.40mm_HandSolder, F.Cu at (101.5, 128.8)
- added R15: 50m, PCM_Resistor_SMD_AKL:R_0805_2012Metric_Pad1.15x1.40mm_HandSolder, B.Cu at (174.6, 117.1)
- added R16: 50m, PCM_Resistor_SMD_AKL:R_0805_2012Metric_Pad1.15x1.40mm_HandSolder, B.Cu at (170.2, 111.5)
- added R17: 50m, PCM_Resistor_SMD_AKL:R_0805_2012Metric_Pad1.15x1.40mm_HandSolder, B.Cu at (160.0, 111.5)
- added R18: 50m, PCM_Resistor_SMD_AKL:R_0805_2012Metric_Pad1.15x1.40mm_HandSolder, B.Cu at (164.5, 117.1)
- added R19: 50m, PCM_Resistor_SMD_AKL:R_0805_2012Metric_Pad1.15x1.40mm_HandSolder, B.Cu at (149.9, 111.5)
- added R20: 50m, PCM_Resistor_SMD_AKL:R_0805_2012Metric_Pad1.15x1.40mm_HandSolder, B.Cu at (154.3, 117.1)
- added R21: 50m, PCM_Resistor_SMD_AKL:R_0805_2012Metric_Pad1.15x1.40mm_HandSolder, B.Cu at (139.7, 111.5)
- added R22: 50m, PCM_Resistor_SMD_AKL:R_0805_2012Metric_Pad1.15x1.40mm_HandSolder, B.Cu at (144.1, 117.1)
- added R7: 1k, Resistor_SMD:R_0805_2012Metric_Pad1.20x1.40mm_HandSolder, F.Cu at (96.8, 122.9)
- added R8: 1k, Resistor_SMD:R_0805_2012Metric_Pad1.20x1.40mm_HandSolder, F.Cu at (96.8, 125.9)
- added R9: 1k, Resistor_SMD:R_0805_2012Metric_Pad1.20x1.40mm_HandSolder, F.Cu at (96.8, 128.8)
- C1, C2: value 10p -> 47p
- J1: value IN+ -> -IN; footprint misc:smd_wire_pad_2.5x5mm -> misc:SMA6251A13GT50G50
- J2: value IN- -> MON; footprint misc:smd_wire_pad_2.5x5mm -> misc:SMA6251A13GT50G50
- J3, J4: footprint misc:smd_wire_pad_2.5x5mm -> misc:726386-2
- J5: value OUT -> GND; footprint misc:smd_wire_pad_2.5x5mm -> misc:726386-2
- J6: value GND -> OUT; footprint misc:smd_wire_pad_2.5x5mm -> misc:726386-2
- Q11: value PZTA42-QX -> MJD31C; footprint Package_TO_SOT_SMD:SOT-223 -> PCM_Package_TO_SOT_SMD_AKL:TO-252-2; moved to B.Cu
- Q12: value PZTA92-QX -> MJD31C; footprint Package_TO_SOT_SMD:SOT-223 -> PCM_Package_TO_SOT_SMD_AKL:TO-252-2; moved to B.Cu
- Q13: value MJD31CG -> MJD31C
- Q14: value MJD32CG -> MJD31C
- Q7, Q8: moved to B.Cu
- R1: value 330k -> 1k
- R2: value 47R -> 330k
- R3: value 47R -> 1k
- R4: value 470R -> 1k
- R5, R6: value 100m -> 1k; footprint PCM_Resistor_SMD_AKL:R_2512_6332Metric_Pad1.40x3.35mm_HandSolder -> Resistor_SMD:R_0805_2012Metric_Pad1.20x1.40mm_HandSolder
- RV1: value 1k -> 500R; footprint misc:G32A_SMD_trimpot -> misc:G43B_SMD_trimpot
- moved J2 83.9 mm to (189.0, 124.5), turned to 90 degrees
- moved J4 67.8 mm to (186.4, 134.6), turned to 90 degrees
- moved C2 57.1 mm to (77.7, 133.7), turned to 0 degrees
- moved J3 54.4 mm to (186.4, 94.0), turned to 90 degrees
- moved R5 50.4 mm to (92.0, 131.8), turned to 0 degrees
- moved C1 50.0 mm to (77.7, 131.2), turned to 0 degrees
- moved RV1 49.8 mm to (78.9, 125.4), turned to 0 degrees
- moved J6 46.6 mm to (186.4, 114.3), turned to 90 degrees
- moved R3 46.5 mm to (92.0, 125.9), turned to 0 degrees
- moved Q8 45.3 mm to (132.1, 135.1), turned to 180 degrees
- moved R6 45.3 mm to (96.8, 120.0), turned to 0 degrees
- moved Q11 43.6 mm to (172.5, 103.8), turned to 90 degrees
- moved Q6 39.0 mm to (87.5, 124.6)
- moved R4 38.5 mm to (92.0, 128.8), turned to 0 degrees
- moved J1 37.0 mm to (90.8, 76.2)
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Connections:
- J1 pad 1: IN+ -> IN-
- J2 pad 1: IN- -> OUT
- J5 pad 1: OUT -> GND
- J6 pad 1: GND -> OUT
- Q11 pad 2: Net-(Q13-C) -> VCC
- Q12 pad 1: Net-(Q12-B) -> Net-(Q11-B)
- Q12 pad 2: Net-(Q14-C) -> VCC
- Q13 pad 1: Net-(Q11-E) -> Net-(Q11-B)
- Q13 pad 2: Net-(Q13-C) -> VCC
- Q13 pad 3: OUT -> Net-(Q13-E)
- Q14 pad 1: Net-(Q12-E) -> Net-(Q11-B)
- Q14 pad 2: Net-(Q14-C) -> VCC
- Q14 pad 3: OUT -> Net-(Q14-E)
- Q7 pad 2: Net-(Q11-B) -> Net-(Q9-B)
- Q7 pad 4: Net-(Q11-B) -> Net-(Q9-B)
- Q8 pad 2: Net-(Q12-B) -> Net-(Q10-B)
- Q8 pad 4: Net-(Q12-B) -> Net-(Q10-B)
- R1 pad 1: Net-(Q2A-B1) -> Net-(Q1B-E2)
- R1 pad 2: Net-(Q1A-B1) -> VCC
- R2 pad 1: Net-(Q7-E) -> Net-(Q2A-B1)
- R2 pad 2: VCC -> Net-(Q1A-B1)
- R3 pad 2: Net-(Q8-E) -> Net-(Q2B-E2)
- R4 pad 1: Net-(R4-Pad1) -> Net-(Q1A-E1)
- R4 pad 2: Net-(Q11-B) -> VCC
- R5 pad 1: Net-(Q13-C) -> VEE
- R5 pad 2: VCC -> Net-(Q2A-E1)
- R6 pad 1: VEE -> Net-(Q5B-E2)
- R6 pad 2: Net-(Q14-C) -> VCC
- RV1 pad 1: Net-(R4-Pad1) -> Net-(R12-Pad1)
- RV1 pad 2: Net-(R4-Pad1) -> Net-(R12-Pad1)
- RV1 pad 3: Net-(Q12-B) -> Net-(Q10-B)
Routing:
- net OUT: track 50.6 -> 0.00 mm, vias 5 -> 0
- net Net-(Q11-B): track 25.1 -> 0.00 mm
- net Net-(Q4A-C1): track 24.6 -> 0.00 mm, vias 3 -> 0
- net Net-(Q12-B): track 20.6 -> 0.00 mm
- net Net-(Q10-B): track 0.00 -> 20.6 mm, vias 0 -> 2
- net Net-(Q3A-C1): track 19.5 -> 0.00 mm, vias 3 -> 0
- net IN-: track 17.7 -> 0.00 mm, vias 2 -> 0
- net Net-(Q10-E): track 0.00 -> 16.0 mm, vias 0 -> 2
- net Net-(Q9-B): track 0.00 -> 14.5 mm
- net IN+: track 13.1 -> 0.00 mm
- net Net-(Q2A-C1): track 12.0 -> 0.00 mm
- net Net-(Q14-C): track 12.0 -> 0.00 mm, vias 4 -> 0
- net Net-(Q13-C): track 12.0 -> 0.00 mm, vias 5 -> 0
- net Net-(Q1A-C1): track 11.9 -> 0.00 mm, vias 2 -> 0
- net Net-(R4-Pad1): track 7.68 -> 0.00 mm
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- added copper zone on B.Cu, net OUT
- added copper zone on B.Cu, net VCC
- added copper zone on B.Cu, net VEE
- removed copper zone on B.Cu, net GND
- removed copper zone on F.Cu, net GND
Other:
- board outline removed
- board text removed: "JLCJLCJLCJLC"
